File: schema_robot_carto/schema_robot_carto.sch (KiCad schematic (older format))
At the start: 9 parts

Commit message: Modif du readme
Parts:
- added R? (x2): R, symbol Device:R
Connections:
- net at J?.32 (PWM0/GPIO12): now also R?.2; no longer Q?.2 (B)
- net at J?.33 (PWM1/GPIO13): now also R?.2; no longer Q?.2 (B)
- new net: Q?.2 (B), R?.1 (x2)
Changed lines of the file:
@@
 	1    0    0    -1
 $EndComp
-$Comp
-L Transistor_BJT:2N2219 Q?
-U 1 1 656E86E5
-P 4600 4450
-F 0 "Q?" H 4790 4496 50  0000 L CNN
-F 1 "2N2219" H 4790 4405 50  0000 L CNN
-F 2 "Package_TO_SOT_THT:TO-39-3" H 4800 4375 50  0001 L CIN
-F 3 "http://www.onsemi.com/pub_link/Collateral/2N2219-D.PDF" H 4600 4450 50  0001 L CNN
-	1    4600 4450
-	1    0    0    -1
-$EndComp
-Wire Wire Line
-	4400 4450 3850 4450
-Wire Wire Line
-	3850 4450 3850 5250
-Wire Wire Line
-	5600 4450 5600 4850
-Wire Wire Line
-	5600 4850 3950 4850
-Wire Wire Line
-	3950 4850 3950 5250
 Wire Wire Line
 	4700 4650 4700 5750
@@
 Wire Wire Line
 	8350 2150 8350 1950
+$Comp
+L Device:R R?
+U 1 1 65887173
+P 3700 4850
+F 0 "R?" H 3770 4896 50  0000 L CNN
+F 1 "R" H 3770 4805 50  0000 L CNN
+F 2 "" V 3630 4850 50  0001 C CNN
+F 3 "~" H 3700 4850 50  0001 C CNN
+	1    3700 4850
+	1    0    0    -1
+$EndComp
+$Comp
+L Device:R R?
+U 1 1 65887774
+P 4100 4850
+F 0 "R?" H 4170 4896 50  0000 L CNN
+F 1 "R" H 4170 4805 50  0000 L CNN
+F 2 "" V 4030 4850 50  0001 C CNN
+F 3 "~" H 4100 4850 50  0001 C CNN
+	1    4100 4850
+	1    0    0    -1
+$EndComp
+$Comp
+L Transistor_BJT:2N2219 Q?
+U 1 1 656E86E5
+P 4600 4450
+F 0 "Q?" H 4790 4496 50  0000 L CNN
+F 1 "2N2219" H 4790 4405 50  0000 L CNN
+F 2 "Package_TO_SOT_THT:TO-39-3" H 4800 4375 50  0001 L CIN
+F 3 "http://www.onsemi.com/pub_link/Collateral/2N2219-D.PDF" H 4600 4450 50  0001 L CNN
+	1    4600 4450
+	1    0    0    -1
+$EndComp
+Wire Wire Line
+	3850 5250 3850 5000
+Wire Wire Line
+	3850 5000 3700 5000
+Wire Wire Line
+	3700 4700 3700 4450
+Wire Wire Line
+	3700 4450 4400 4450
+Wire Wire Line
+	3950 5250 4100 5250
+Wire Wire Line
+	4100 5250 4100 5000
+Wire Wire Line
+	4100 4700 5600 4700
+Wire Wire Line
+	5600 4700 5600 4450
 $EndSCHEMATC

Commit message: mise à jour des schémas et README
Parts:
- removed M? (x2): Motor_DC, symbol Motor:Motor_DC
- removed Q? (x2): 2N2219, Package_TO_SOT_THT:TO-39-3, symbol Transistor_BJT:2N2219
- removed R? (x2): R, symbol Device:R
- added M? (x2): Motor_DC, symbol Motor:Motor_DC
- added U?: L298HN, Package_TO_SOT_THT:TO-220-15_P2.54x2.54mm_StaggerOdd_Lead4.58mm_Vertical, symbol Driver_Motor:L298HN
- gave numbers to parts that had none: 1
Connections:
- net +3V8: now also RASPBERRY_PI_ZERO.21 (MISO0/GPIO9), U?.7 (IN2)
- net at RASPBERRY_PI_ZERO.19 (MOSI0/GPIO10): now also U?.10 (IN3)
- net +5V: now reaches RASPBERRY_PI_ZERO.2 (5V)
- net +5V: now also U?.9 (Vss)
- net at RASPBERRY_PI_ZERO.23 (SCLK0/GPIO11): now also U?.12 (IN4)
- net at RASPBERRY_PI_ZERO.24 (~CE0~/GPIO8): now also U?.5 (IN1)
- net at RASPBERRY_PI_ZERO.32 (PWM0/GPIO12): now also U?.6 (EnA)
- net at RASPBERRY_PI_ZERO.33 (PWM1/GPIO13): now also U?.11 (EnB)
- net at RASPBERRY_PI_ZERO.39 (GND): now also U?.8 (GND)
- new net: M?.2 (-), U?.13 (OUT3)
- new net: M?.1 (+), U?.14 (OUT4)
- new net: M?.1 (+), U?.3 (OUT2)
- new net +8V: U?.4 (Vs)
Changed lines of the file:
@@
 	7050 2150 7150 2150
-$Comp
-L Motor:Motor_DC M?
-U 1 1 656E63B0
-P 4700 3600
-F 0 "M?" H 4858 3596 50  0000 L CNN
-F 1 "Motor_DC" H 4858 3505 50  0000 L CNN
-F 2 "" H 4700 3510 50  0001 C CNN
-F 3 "~" H 4700 3510 50  0001 C CNN
-	1    4700 3600
-	1    0    0    -1
-$EndComp
-Wire Wire Line
-	4700 4650 4700 5750
-Connection ~ 4700 5750
-Wire Wire Line
-	6100 4650 6100 5750
-Wire Wire Line
-	5800 4450 5600 4450
-$Comp
-L Transistor_BJT:2N2219 Q?
-U 1 1 656F3E9E
-P 6000 4450
-F 0 "Q?" H 6190 4496 50  0000 L CNN
-F 1 "2N2219" H 6190 4405 50  0000 L CNN
-F 2 "Package_TO_SOT_THT:TO-39-3" H 6200 4375 50  0001 L CIN
-F 3 "http://www.onsemi.com/pub_link/Collateral/2N2219-D.PDF" H 6000 4450 50  0001 L CNN
-	1    6000 4450
-	1    0    0    -1
-$EndComp
-$Comp
-L Motor:Motor_DC M?
-U 1 1 656E6BB4
-P 6100 3600
-F 0 "M?" H 6258 3596 50  0000 L CNN
-F 1 "Motor_DC" H 6258 3505 50  0000 L CNN
-F 2 "" H 6100 3510 50  0001 C CNN
-F 3 "~" H 6100 3510 50  0001 C CNN
-	1    6100 3600
-	1    0    0    -1
-$EndComp
 $Comp
 L power:+3V8 #PWR?
@@
 	1    0    0    -1
 $EndComp
-Wire Wire Line
-	4700 3400 5450 3400
-Wire Wire Line
-	5450 3400 5450 3200
-Wire Wire Line
-	6100 3400 5450 3400
-Connection ~ 5450 3400
-Wire Wire Line
-	4700 3900 4700 4250
-Wire Wire Line
-	6100 3900 6100 4250
-Wire Wire Line
-	6100 5750 4700 5750
-Wire Wire Line
-	4700 5750 4450 5750
-$Comp
-L Connector:Raspberry_Pi_2_3 J?
+$Comp
+L Connector:Raspberry_Pi_2_3 RASPBERRY_PI_ZERO
 U 1 1 656D6484
 P 3150 6050
-F 0 "J?" V 3196 7394 50  0000 L CNN
+F 0 "RASPBERRY_PI_ZERO" V 3196 7394 50  0000 L CNN
 F 1 "Raspberry_Pi_2_3" V 3105 7394 50  0000 L CNN
 F 2 "" H 3150 6050 50  0001 C CNN
@@
 Wire Wire Line
 	8350 2150 8350 1950
-$Comp
-L Device:R R?
-U 1 1 65887173
-P 3700 4850
-F 0 "R?" H 3770 4896 50  0000 L CNN
-F 1 "R" H 3770 4805 50  0000 L CNN
-F 2 "" V 3630 4850 50  0001 C CNN
-F 3 "~" H 3700 4850 50  0001 C CNN
-	1    3700 4850
-	1    0    0    -1
-$EndComp
-$Comp
-L Device:R R?
-U 1 1 65887774
-P 4100 4850
-F 0 "R?" H 4170 4896 50  0000 L CNN
-F 1 "R" H 4170 4805 50  0000 L CNN
-F 2 "" V 4030 4850 50  0001 C CNN
-F 3 "~" H 4100 4850 50  0001 C CNN
-	1    4100 4850
-	1    0    0    -1
-$EndComp
-$Comp
-L Transistor_BJT:2N2219 Q?
-U 1 1 656E86E5
-P 4600 4450
-F 0 "Q?" H 4790 4496 50  0000 L CNN
-F 1 "2N2219" H 4790 4405 50  0000 L CNN
-F 2 "Package_TO_SOT_THT:TO-39-3" H 4800 4375 50  0001 L CIN
-F 3 "http://www.onsemi.com/pub_link/Collateral/2N2219-D.PDF" H 4600 4450 50  0001 L CNN
-	1    4600 4450
-	1    0    0    -1
-$EndComp
-Wire Wire Line
-	3850 5250 3850 5000
-Wire Wire Line
-	3850 5000 3700 5000
-Wire Wire Line
-	3700 4700 3700 4450
-Wire Wire Line
-	3700 4450 4400 4450
 Wire Wire Line
 	3950 5250 4100 5250
-Wire Wire Line
-	4100 5250 4100 5000
-Wire Wire Line
-	4100 4700 5600 4700
-Wire Wire Line
-	5600 4700 5600 4450
+$Comp
+L Driver_Motor:L298HN U?
+U 1 1 659DE89E
+P 5850 4400
+F 0 "U?" V 5804 5144 50  0000 L CNN
+F 1 "L298HN" V 5895 5144 50  0000 L CNN
+F 2 "Package_TO_SOT_THT:TO-220-15_P2.54x2.54mm_StaggerOdd_Lead4.58mm_Vertical" H 5900 3750 50  0001 L CNN
+F 3 "http://www.st.com/st-web-ui/static/active/en/resource/technical/document/datasheet/CD00000240.pdf" H 6000 4650 50  0001 C CNN
+	1    5850 4400
+	0    1    1    0
+$EndComp
+$Comp
+L Motor:Motor_DC M?
+U 1 1 659DFA11
+P 5300 5650
+F 0 "M?" H 5458 5646 50  0000 L CNN
+F 1 "Motor_DC" H 5458 5555 50  0000 L CNN
+F 2 "" H 5300 5560 50  0001 C CNN
+F 3 "~" H 5300 5560 50  0001 C CNN
+	1    5300 5650
+	0    -1   -1   0
+$EndComp
+$Comp
+L Motor:Motor_DC M?
+U 1 1 659E00C8
+P 6300 5650
+F 0 "M?" H 6458 5646 50  0000 L CNN
+F 1 "Motor_DC" H 6458 5555 50  0000 L CNN
+F 2 "" H 6300 5560 50  0001 C CNN
+F 3 "~" H 6300 5560 50  0001 C CNN
+	1    6300 5650
+	0    -1   -1   0
+$EndComp
+Wire Wire Line
+	5600 5650 5600 5350
+Wire Wire Line
+	5600 5350 5750 5350
+Wire Wire Line
+	5750 5350 5750 5000
+Wire Wire Line
+	5100 5650 5100 5150
+Wire Wire Line
+	5100 5150 5650 5150
+Wire Wire Line
+	5650 5150 5650 5000
+Wire Wire Line
+	6100 5650 6100 5250
+Wire Wire Line
+	6100 5250 5950 5250
+Wire Wire Line
+	5950 5250 5950 5000
+Wire Wire Line
+	6600 5600 6600 5100
+Wire Wire Line
+	6600 5100 6050 5100
+Wire Wire Line
+	6050 5100 6050 5000
+Wire Wire Line
+	4100 3600 5750 3600
+Wire Wire Line
+	5750 3600 5750 3800
+Wire Wire Line
+	4100 3600 4100 5250
+Wire Wire Line
+	3650 5250 3650 4350
+Wire Wire Line
+	3650 4350 5050 4350
+Wire Wire Line
+	5050 4350 5050 3300
+Wire Wire Line
+	5050 3300 5850 3300
+Wire Wire Line
+	5850 3300 5850 3800
+Wire Wire Line
+	3550 5250 3550 4300
+Wire Wire Line
+	3550 4300 5000 4300
+Wire Wire Line
+	5000 4300 5000 3250
+Wire Wire Line
+	5000 3250 5950 3250
+Wire Wire Line
+	5950 3250 5950 3800
+Wire Wire Line
+	3450 5250 3450 4250
+Wire Wire Line
+	3450 4250 4950 4250
+Wire Wire Line
+	4950 4250 4950 3200
+Wire Wire Line
+	4950 3200 5450 3200
+Wire Wire Line
+	6250 3200 6250 3800
+Connection ~ 5450 3200
+Wire Wire Line
+	5450 3200 6250 3200
+Wire Wire Line
+	3350 5250 3350 4200
+Wire Wire Line
+	3350 4200 4900 4200
+Wire Wire Line
+	4900 4200 4900 3150
+Wire Wire Line
+	4900 3150 6350 3150
+Wire Wire Line
+	6350 3150 6350 3800
+Wire Wire Line
+	6150 3550 4050 3550
+Wire Wire Line
+	4050 3550 4050 5200
+Wire Wire Line
+	4050 5200 3850 5200
+Wire Wire Line
+	3850 5200 3850 5250
+Wire Wire Line
+	6150 3550 6150 3800
+Wire Wire Line
+	5150 4400 5150 4900
+Wire Wire Line
+	5150 4900 4450 4900
+Wire Wire Line
+	4450 4900 4450 5750
+$Comp
+L power:+8V #PWR?
+U 1 1 65A10A30
+P 6750 4500
+F 0 "#PWR?" H 6750 4350 50  0001 C CNN
+F 1 "+8V" V 6765 4628 50  0000 L CNN
+F 2 "" H 6750 4500 50  0001 C CNN
+F 3 "" H 6750 4500 50  0001 C CNN
+	1    6750 4500
+	0    1    1    0
+$EndComp
+Wire Wire Line
+	6550 4500 6750 4500
+Wire Wire Line
+	6550 4400 7250 4400
+Wire Wire Line
+	7250 4400 7250 6300
+Wire Wire Line
+	7250 6300 5000 6300
+Wire Wire Line
+	5000 6300 5000 7100
+Wire Wire Line
+	5000 7100 1850 7100
+Wire Wire Line
+	1850 7100 1850 6250
+$Comp
+L power:+5V #PWR?
+U 1 1 65A17912
+P 7250 4400
+F 0 "#PWR?" H 7250 4250 50  0001 C CNN
+F 1 "+5V" H 7265 4573 50  0000 C CNN
+F 2 "" H 7250 4400 50  0001 C CNN
+F 3 "" H 7250 4400 50  0001 C CNN
+	1    7250 4400
+	1    0    0    -1
+$EndComp
+Connection ~ 7250 4400
 $EndSCHEMATC
